File: magnetophone.sch (EAGLE design)
At the start: 22 parts, among them U1 TL074_

Commit message: double!
Parts:
- added C7: 47uf, SparkFun-Passives:CAP_POLPTH2
- added C8: 15nf, TomW:C-EU050-024X044
- added GAIN1: 50k, TomW:ALPHA-9MMF2A
- added R2, R6: 2.2k, TomW:R-EU_STANDARD_RESISTOR
- added R3: 220R, TomW:R-EU_STANDARD_RESISTOR
- added R4: 200R, TomW:R-EU_STANDARD_RESISTOR
- added R5: 200k, TomW:R-EU_STANDARD_RESISTOR
- added R7: 3.6k, TomW:R-EU_STANDARD_RESISTOR
- added RV1: (no value), SparkFun-Electromechanical:POT_DUAL
- added U$4: MONO_CASSETTE_HEAD, MusicThingModular:MONO_CASSETTE_HEAD
- added U$5, U$6: THONKICONNNEW, MusicThingModular:THONKICONNNEW
Connections:
- new net N$11: U$5.TIP, U1C.+IN
- new net N$12: GAIN1.E, GAIN1.S, R3.1, U1D.OUT
- new net N$13: R3.2, U$6.TIP
- new net N$14: R5.1, R7.2, U1C.OUT, U1D.+IN
- new net N$15: C8.2, R4.2, R5.2, U1C.-IN
- new net N$16: R2.2, R6.2, U1D.-IN
- new net N$17: GAIN1.A, R2.1
- new net N$18: U$4.P$1, U$5.SWITCH
- new net N$19: C7.+, R4.1
- new net N$20: C8.1, R7.1
- net GND: now also C7.-, R6.1, U$4.P$2, U$5.SLEEVE, U$6.SLEEVE
Other:
- moved on the sheet: U1C, U1D
Changed lines of the file:
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@@
 <part name="U$2" library="MusicThingModular" deviceset="THONKICONN" device="NEW"/>
 <part name="U$3" library="MusicThingModular" deviceset="THONKICONN" device="NEW"/>
+<part name="RV1" library="SparkFun-Electromechanical" deviceset="POT_DUAL" device=""/>
+<part name="GAIN1" library="TomW" deviceset="ALPHA-9MM" device="A" technology="F2" value="50k"/>
+<part name="SUPPLY2" library="supply2" deviceset="GND" device=""/>
+<part name="R2" library="TomW" deviceset="R-EU_" device="STANDARD_RESISTOR" value="2.2k"/>
+<part name="R3" library="TomW" deviceset="R-EU_" device="STANDARD_RESISTOR" value="220R"/>
+<part name="SUPPLY4" library="supply2" deviceset="GND" device=""/>
+<part name="R4" library="TomW" deviceset="R-EU_" device="STANDARD_RESISTOR" value="200R"/>
+<part name="R5" library="TomW" deviceset="R-EU_" device="STANDARD_RESISTOR" value="200k"/>
+<part name="SUPPLY6" library="supply2" deviceset="GND" device=""/>
+<part name="R6" library="TomW" deviceset="R-EU_" device="STANDARD_RESISTOR" value="2.2k"/>
+<part name="SUPPLY8" library="supply2" deviceset="GND" device=""/>
+<part name="U$4" library="MusicThingModular" deviceset="MONO_CASSETTE_HEAD" device=""/>
+<part name="SUPPLY10" library="supply2" deviceset="GND" device=""/>
+<part name="C7" library="SparkFun-Passives" deviceset="CAP_POL" device="PTH2" value="47uf"/>
+<part name="C8" library="TomW" deviceset="C-EU" device="050-024X044" value="15nf"/>
+<part name="R7" library="TomW" deviceset="R-EU_" device="STANDARD_RESISTOR" value="3.6k"/>
+<part name="U$5" library="MusicThingModular" deviceset="THONKICONN" device="NEW"/>
+<part name="U$6" library="MusicThingModular" deviceset="THONKICONN" device="NEW"/>
 </parts>
 <sheets>
@@
 fuses with jumper wire.
 Don't get it the wrong way around! </text>
+<text x="355.6" y="147.32" size="1.778" layer="91">NAB Equalisation and
+first gain stage
+100 - 1000x gain
+according to freq
+ </text>
+<text x="393.7" y="147.32" size="1.778" layer="91">Non inverting stage
+1-26 x gain
+Total gain =  5-130 </text>
 </plain>
 <instances>
@@
 <instance part="U$1" gate="G$1" x="45.72" y="116.84"/>
 <instance part="SUPPLY1" gate="GND" x="55.88" y="109.22"/>
-<instance part="U1" gate="C" x="218.44" y="91.44"/>
-<instance part="U1" gate="D" x="238.76" y="88.9"/>
+<instance part="U1" gate="C" x="365.76" y="137.16"/>
+<instance part="U1" gate="D" x="401.32" y="137.16"/>
 <instance part="U1" gate="P" x="124.46" y="66.04"/>
 <instance part="C3" gate="G$1" x="116.84" y="88.9"/>
@@
 <instance part="U$2" gate="G$1" x="71.12" y="119.38"/>
 <instance part="U$3" gate="G$1" x="205.74" y="124.46"/>
+<instance part="RV1" gate="G$1" x="190.5" y="101.6"/>
+<instance part="RV1" gate="G$2" x="243.84" y="119.38"/>
+<instance part="GAIN1" gate="G$1" x="414.02" y="116.84"/>
+<instance part="SUPPLY2" gate="GND" x="302.26" y="119.38"/>
+<instance part="R2" gate="G$1" x="403.86" y="124.46" rot="R180"/>
+<instance part="R3" gate="G$1" x="426.72" y="137.16"/>
+<instance part="SUPPLY4" gate="GND" x="436.88" y="127"/>
+<instance part="R4" gate="G$1" x="353.06" y="109.22" rot="R90"/>
+<instance part="R5" gate="G$1" x="363.22" y="116.84" rot="R180"/>
+<instance part="SUPPLY6" gate="GND" x="353.06" y="88.9"/>
+<instance part="R6" gate="G$1" x="393.7" y="114.3" rot="R90"/>
+<instance part="SUPPLY8" gate="GND" x="393.7" y="106.68"/>
+<instance part="U$4" gate="G$1" x="281.94" y="127"/>
+<instance part="SUPPLY10" gate="GND" x="292.1" y="119.38"/>
+<instance part="C7" gate="G$1" x="353.06" y="99.06"/>
+<instance part="C8" gate="G$1" x="360.68" y="127" rot="R270"/>
+<instance part="R7" gate="G$1" x="370.84" y="127"/>
+<instance part="U$5" gate="G$1" x="307.34" y="129.54"/>
+<instance part="U$6" gate="G$1" x="441.96" y="134.62"/>
 </instances>
 <busses>
@@
 <pinref part="SUPPLY9" gate="GND" pin="GND"/>
 <wire x1="116.84" y1="83.82" x2="116.84" y2="81.28" width="0.1524" layer="91"/>
+</segment>
+<segment>
+<wire x1="302.26" y1="127" x2="302.26" y2="121.92" width="0.1524" layer="91"/>
+<pinref part="SUPPLY2" gate="GND" pin="GND"/>
+<pinref part="U$5" gate="G$1" pin="SLEEVE"/>
+</segment>
+<segment>
+<pinref part="SUPPLY4" gate="GND" pin="GND"/>
+<wire x1="436.88" y1="129.54" x2="436.88" y2="132.08" width="0.1524" layer="91"/>
+<pinref part="U$6" gate="G$1" pin="SLEEVE"/>
+</segment>
+<segment>
+<pinref part="R6" gate="G$1" pin="1"/>
+<pinref part="SUPPLY8" gate="GND" pin="GND"/>
+</segment>
+<segment>
+<pinref part="U$4" gate="G$1" pin="P$2"/>
+<pinref part="SUPPLY10" gate="GND" pin="GND"/>
+<wire x1="289.56" y1="124.46" x2="292.1" y2="124.46" width="0.1524" layer="91"/>
+<wire x1="292.1" y1="124.46" x2="292.1" y2="121.92" width="0.1524" layer="91"/>
+</segment>
+<segment>
+<pinref part="C7" gate="G$1" pin="-"/>
+<pinref part="SUPPLY6" gate="GND" pin="GND"/>
+<wire x1="353.06" y1="93.98" x2="353.06" y2="91.44" width="0.1524" layer="91"/>
 </segment>
 </net>
@@
 </segment>
 </net>
+<net name="N$11" class="0">
+<segment>
+<wire x1="302.26" y1="132.08" x2="302.26" y2="139.7" width="0.1524" layer="91"/>
+<wire x1="302.26" y1="139.7" x2="358.14" y2="139.7" width="0.1524" layer="91"/>
+<pinref part="U$5" gate="G$1" pin="TIP"/>
+<pinref part="U1" gate="C" pin="+IN"/>
+</segment>
+</net>
+<net name="N$12" class="0">
+<segment>
+<wire x1="421.64" y1="137.16" x2="419.1" y2="137.16" width="0.1524" layer="91"/>
+<wire x1="419.1" y1="137.16" x2="408.94" y2="137.16" width="0.1524" layer="91"/>
+<pinref part="R3" gate="G$1" pin="1"/>
+<pinref part="GAIN1" gate="G$1" pin="S"/>
+<wire x1="419.1" y1="137.16" x2="419.1" y2="124.46" width="0.1524" layer="91"/>
+<junction x="419.1" y="137.16"/>
+<pinref part="GAIN1" gate="G$1" pin="E"/>
+<wire x1="419.1" y1="124.46" x2="419.1" y2="116.84" width="0.1524" layer="91"/>
+<wire x1="414.02" y1="124.46" x2="419.1" y2="124.46" width="0.1524" layer="91"/>
+<junction x="419.1" y="124.46"/>
+<pinref part="U1" gate="D" pin="OUT"/>
+</segment>
+</net>
+<net name="N$13" class="0">
+<segment>
+<pinref part="R3" gate="G$1" pin="2"/>
+<wire x1="436.88" y1="137.16" x2="431.8" y2="137.16" width="0.1524" layer="91"/>
+<pinref part="U$6" gate="G$1" pin="TIP"/>
+</segment>
+</net>
+<net name="N$14" class="0">
+<segment>
+<wire x1="373.38" y1="137.16" x2="378.46" y2="137.16" width="0.1524" layer="91"/>
+<wire x1="378.46" y1="137.16" x2="378.46" y2="127" width="0.1524" layer="91"/>
+<junction x="378.46" y="137.16"/>
+<pinref part="R5" gate="G$1" pin="1"/>
+<wire x1="378.46" y1="127" x2="378.46" y2="116.84" width="0.1524" layer="91"/>
+<wire x1="368.3" y1="116.84" x2="378.46" y2="116.84" width="0.1524" layer="91"/>
+<wire x1="378.46" y1="137.16" x2="378.46" y2="139.7" width="0.1524" layer="91"/>
+<wire x1="378.46" y1="139.7" x2="393.7" y2="139.7" width="0.1524" layer="91"/>
+<pinref part="R7" gate="G$1" pin="2"/>
+<wire x1="375.92" y1="127" x2="378.46" y2="127" width="0.1524" layer="91"/>
+<junction x="378.46" y="127"/>
+<pinref part="U1" gate="C" pin="OUT"/>
+<pinref part="U1" gate="D" pin="+IN"/>
+</segment>
+</net>
+<net name="N$15" class="0">
+<segment>
+<wire x1="353.06" y1="116.84" x2="353.06" y2="127" width="0.1524" layer="91"/>
+<wire x1="353.06" y1="127" x2="353.06" y2="134.62" width="0.1524" layer="91"/>
+<wire x1="353.06" y1="134.62" x2="358.14" y2="134.62" width="0.1524" layer="91"/>
+<pinref part="R5" gate="G$1" pin="2"/>
+<wire x1="358.14" y1="116.84" x2="353.06" y2="116.84" width="0.1524" layer="91"/>
+<pinref part="R4" gate="G$1" pin="2"/>
+<wire x1="353.06" y1="114.3" x2="353.06" y2="116.84" width="0.1524" layer="91"/>
+<junction x="353.06" y="116.84"/>
+<pinref part="C8" gate="G$1" pin="2"/>
+<wire x1="355.6" y1="127" x2="353.06" y2="127" width="0.1524" layer="91"/>
+<junction x="353.06" y="127"/>
+<pinref part="U1" gate="C" pin="-IN"/>
+</segment>
+</net>
+<net name="N$16" class="0">
+<segment>
+<wire x1="393.7" y1="134.62" x2="393.7" y2="124.46" width="0.1524" layer="91"/>
+<pinref part="R6" gate="G$1" pin="2"/>
+<pinref part="R2" gate="G$1" pin="2"/>
+<wire x1="393.7" y1="124.46" x2="393.7" y2="119.38" width="0.1524" layer="91"/>
+<wire x1="398.78" y1="124.46" x2="393.7" y2="124.46" width="0.1524" layer="91"/>
+<junction x="393.7" y="124.46"/>
+<pinref part="U1" gate="D" pin="-IN"/>
+</segment>
+</net>
+<net name="N$17" class="0">
+<segment>
+<pinref part="R2" gate="G$1" pin="1"/>
+<wire x1="408.94" y1="124.46" x2="408.94" y2="109.22" width="0.1524" layer="91"/>
+<pinref part="GAIN1" gate="G$1" pin="A"/>
+<wire x1="408.94" y1="109.22" x2="414.02" y2="109.22" width="0.1524" layer="91"/>
+</segment>
+</net>
+<net name="N$18" class="0">
+<segment>
+<pinref part="U$4" gate="G$1" pin="P$1"/>
+<wire x1="289.56" y1="129.54" x2="302.26" y2="129.54" width="0.1524" layer="91"/>
+<pinref part="U$5" gate="G$1" pin="SWITCH"/>
+</segment>
+</net>
+<net name="N$19" class="0">
+<segment>
+<pinref part="C7" gate="G$1" pin="+"/>
+<pinref part="R4" gate="G$1" pin="1"/>
+<wire x1="353.06" y1="101.6" x2="353.06" y2="104.14" width="0.1524" layer="91"/>
+</segment>
+</net>
+<net name="N$20" class="0">
+<segment>
+<pinref part="C8" gate="G$1" pin="1"/>
+<pinref part="R7" gate="G$1" pin="1"/>
+<wire x1="363.22" y1="127" x2="365.76" y2="127" width="0.1524" layer="91"/>
+</segment>
+</net>

Commit message: Starting layout
Parts:
- removed C7: 47uf, SparkFun-Passives:CAP_POLPTH2
- removed C8: 15nf, TomW:C-EU050-024X044
- removed GAIN1: 50k, TomW:ALPHA-9MMF2A
- removed R2, R6: 2.2k, TomW:R-EU_STANDARD_RESISTOR
- removed R3: 220R, TomW:R-EU_STANDARD_RESISTOR
- removed R4: 200R, TomW:R-EU_STANDARD_RESISTOR
- removed R5: 200k, TomW:R-EU_STANDARD_RESISTOR
- removed R7: 3.6k, TomW:R-EU_STANDARD_RESISTOR
- removed RV1: (no value), SparkFun-Electromechanical:POT_DUAL
- removed U$4: MONO_CASSETTE_HEAD, MusicThingModular:MONO_CASSETTE_HEAD
- removed U$5, U$6: THONKICONNNEW, MusicThingModular:THONKICONNNEW
- removed U1: TL074_, MusicThingModular:TL074_
- added U2: TL072_, MusicThingModular:TL072_
- R1, R10, R12, R14, R16, R8: device TomW:R-EU_STANDARD_RESISTOR -> MusicThingModular:RESISTOR7MM
- renumbered U$2 to EXT, U$3 to OUT
Connections:
- removed net N$11: U$5.TIP, U1C.+IN
- removed net N$12: GAIN1.E, GAIN1.S, R3.1, U1D.OUT
- removed net N$13: R3.2, U$6.TIP
- removed net N$14: R5.1, R7.2, U1C.OUT, U1D.+IN
- removed net N$15: C8.2, R4.2, R5.2, U1C.-IN
- removed net N$16: R2.2, R6.2, U1D.-IN
- removed net N$17: GAIN1.A, R2.1
- removed net N$18: U$4.P$1, U$5.SWITCH
- removed net N$19: C7.+, R4.1
- removed net N$20: C8.1, R7.1
- net +12V: now also U2P.V+; no longer U1P.V+
- net -12V: now also U2P.V-; no longer U1P.V-
- net GND: now also R12.2; no longer C7.-, R12.1, R6.1, U$4.P$2, U$5.SLEEVE, U$6.SLEEVE
- net N$2: now also U2A.+IN; no longer U1A.+IN
- net N$3: now also R10.1, R8.1, U2A.-IN; no longer R10.2, R8.2, U1A.-IN
- net N$4: now also R10.2, U2A.OUT, U2B.+IN; no longer R10.1, U1A.OUT, U1B.+IN
- net N$6: now also R12.1, U2B.-IN; no longer R12.2, U1B.-IN
- net N$7: now also R8.2; no longer R8.1
- net N$8: now also U2B.OUT; no longer U1B.OUT
Other:
- moved on the sheet: R10, R12, R8

Commit message: First pcb layout
Parts:
- removed SV1: (no value), TomW:10_PIN_HEADER
- added U$2: EURO_POWER_LOCK, MusicThingModular:EURO_POWER_LOCK
Connections:
- net +12V_INLET: now also U$2.+12V; no longer SV1.10, SV1.9
- net -12V: now also C5.1; no longer C5.2
- net -12V_INLET: now also U$2.-12V; no longer SV1.1, SV1.2
- net GND: now also C5.2, R12.1, U$2.GND; no longer C5.1, R12.2, SV1.3, SV1.4, SV1.5, SV1.6, SV1.7, SV1.8
- net N$10: now also R16.1; no longer R16.2
- net N$6: now also R12.2; no longer R12.1
- net N$8: now also R16.2; no longer R16.1
Changed lines of the file:
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@@
 <?xml version="1.0" encoding="utf-8"?>
 <!DOCTYPE eagle SYSTEM "eagle.dtd">
-<eagle version="7.2.0">
+<eagle version="7.4.0">
 <drawing>
 <settings>
@@
 </variantdefs>
 <classes>
-<class number="0" name="default" width="0.6096" drill="0">
+<class number="0" name="default" width="0.3048" drill="0">
 </class>
 <class number="1" name="power" width="0.6096" drill="0">
@@
 <parts>
 <part name="GAIN" library="TomW" deviceset="ALPHA-9MM" device="A" technology="F2" value="50k"/>
-<part name="SV1" library="TomW" deviceset="10_PIN_HEADER" device=""/>
 <part name="SUPPLY3" library="supply2" deviceset="GND" device=""/>
 <part name="R14" library="MusicThingModular" deviceset="RESISTOR" device="7MM" value="2.2k"/>
@@
 <part name="OUT" library="MusicThingModular" deviceset="THONKICONN" device="NEW"/>
 <part name="U2" library="MusicThingModular" deviceset="TL072" device="_"/>
+<part name="U$2" library="MusicThingModular" deviceset="EURO_POWER_LOCK" device=""/>
 </parts>
 <sheets>
@@
 <instance part="U2" gate="B" x="165.1" y="127"/>
 <instance part="GAIN" gate="G$1" x="177.8" y="106.68"/>
-<instance part="SV1" gate="G$1" x="71.12" y="60.96"/>
 <instance part="SUPPLY3" gate="GND" x="66.04" y="109.22"/>
 <instance part="R14" gate="G$1" x="167.64" y="114.3" rot="R180"/>
@@
 <instance part="OUT" gate="G$1" x="205.74" y="124.46"/>
 <instance part="U2" gate="P" x="124.46" y="66.04"/>
+<instance part="U$2" gate="G$1" x="73.66" y="60.96"/>
 </instances>
 <busses>
@@
 <net name="GND" class="2">
 <segment>
-<pinref part="SV1" gate="G$1" pin="7"/>
-<wire x1="81.28" y1="63.5" x2="78.74" y2="63.5" width="0.1524" layer="91"/>
-<label x="81.28" y="63.5" size="1.778" layer="95"/>
-</segment>
-<segment>
-<pinref part="SV1" gate="G$1" pin="5"/>
 <wire x1="81.28" y1="60.96" x2="78.74" y2="60.96" width="0.1524" layer="91"/>
 <label x="81.28" y="60.96" size="1.778" layer="95"/>
-</segment>
-<segment>
-<pinref part="SV1" gate="G$1" pin="3"/>
-<wire x1="81.28" y1="58.42" x2="78.74" y2="58.42" width="0.1524" layer="91"/>
-<label x="81.28" y="58.42" size="1.778" layer="95"/>
-</segment>
-<segment>
-<pinref part="SV1" gate="G$1" pin="8"/>
-<wire x1="60.96" y1="63.5" x2="63.5" y2="63.5" width="0.1524" layer="91"/>
-<label x="58.42" y="63.5" size="1.778" layer="95"/>
-</segment>
-<segment>
-<pinref part="SV1" gate="G$1" pin="6"/>
-<wire x1="60.96" y1="60.96" x2="63.5" y2="60.96" width="0.1524" layer="91"/>
-<label x="58.42" y="60.96" size="1.778" layer="95"/>
-</segment>
-<segment>
-<pinref part="SV1" gate="G$1" pin="4"/>
-<wire x1="60.96" y1="58.42" x2="63.5" y2="58.42" width="0.1524" layer="91"/>
-<label x="58.42" y="58.42" size="1.778" layer="95"/>
+<pinref part="U$2" gate="G$1" pin="GND"/>
 </segment>
 <segment>
@@
 </segment>
 <segment>
-<pinref part="R12" gate="G$1" pin="2"/>
+<pinref part="R12" gate="G$1" pin="1"/>
 <pinref part="SUPPLY5" gate="GND" pin="GND"/>
+<wire x1="157.48" y1="99.06" x2="157.48" y2="109.22" width="0.1524" layer="91"/>
 </segment>
 <segment>
@@
 </segment>
 <segment>
-<wire x1="132.08" y1="63.5" x2="132.08" y2="66.04" width="0.1524" layer="91"/>
+<wire x1="132.08" y1="55.88" x2="132.08" y2="66.04" width="0.1524" layer="91"/>
 <wire x1="132.08" y1="66.04" x2="142.24" y2="66.04" width="0.1524" layer="91"/>
 <pinref part="GND22" gate="1" pin="GND"/>
 <pinref part="C4" gate="G$1" pin="2"/>
 <junction x="132.08" y="66.04"/>
-<pinref part="C5" gate="G$1" pin="1"/>
+<pinref part="C5" gate="G$1" pin="2"/>
 </segment>
 <segment>
@@
 <segment>
 <pinref part="SUPPLY18" gate="G$1" pin="-12V"/>
-<pinref part="C5" gate="G$1" pin="2"/>
+<pinref part="C5" gate="G$1" pin="1"/>
 <wire x1="132.08" y1="52.07" x2="132.08" y2="53.34" width="0.1524" layer="91"/>
-<wire x1="132.08" y1="53.34" x2="132.08" y2="55.88" width="0.1524" layer="91"/>
+<wire x1="132.08" y1="53.34" x2="132.08" y2="63.5" width="0.1524" layer="91"/>
 <wire x1="124.46" y1="58.42" x2="124.46" y2="53.34" width="0.1524" layer="91"/>
 <wire x1="124.46" y1="53.34" x2="132.08" y2="53.34" width="0.1524" layer="91"/>
@@
 <segment>
 <pinref part="U2" gate="B" pin="OUT"/>
-<wire x1="185.42" y1="127" x2="182.88" y2="127" width="0.1524" layer="91"/>
+<wire x1="195.58" y1="127" x2="182.88" y2="127" width="0.1524" layer="91"/>
 <wire x1="182.88" y1="127" x2="172.72" y2="127" width="0.1524" layer="91"/>
-<pinref part="R16" gate="G$1" pin="1"/>
+<pinref part="R16" gate="G$1" pin="2"/>
 <pinref part="GAIN" gate="G$1" pin="S"/>
 <wire x1="182.88" y1="127" x2="182.88" y2="114.3" width="0.1524" layer="91"/>
@@
 <net name="N$10" class="0">
 <segment>
-<pinref part="R16" gate="G$1" pin="2"/>
-<wire x1="200.66" y1="127" x2="195.58" y2="127" width="0.1524" layer="91"/>
+<pinref part="R16" gate="G$1" pin="1"/>
+<wire x1="200.66" y1="127" x2="185.42" y2="127" width="0.1524" layer="91"/>
 <pinref part="OUT" gate="G$1" pin="TIP"/>
 </segment>
@@
 <pinref part="U2" gate="B" pin="-IN"/>
 <wire x1="157.48" y1="124.46" x2="157.48" y2="114.3" width="0.1524" layer="91"/>
-<pinref part="R12" gate="G$1" pin="1"/>
+<pinref part="R12" gate="G$1" pin="2"/>
 <pinref part="R14" gate="G$1" pin="2"/>
-<wire x1="157.48" y1="114.3" x2="157.48" y2="109.22" width="0.1524" layer="91"/>
+<wire x1="157.48" y1="114.3" x2="157.48" y2="99.06" width="0.1524" layer="91"/>
 <wire x1="162.56" y1="114.3" x2="157.48" y2="114.3" width="0.1524" layer="91"/>
 <junction x="157.48" y="114.3"/>
@@
 <net name="+12V_INLET" class="0">
 <segment>
-<pinref part="SV1" gate="G$1" pin="10"/>
-<wire x1="60.96" y1="66.04" x2="63.5" y2="66.04" width="0.1524" layer="91"/>
-<label x="45.72" y="66.04" size="1.778" layer="95"/>
-</segment>
-<segment>
-<pinref part="SV1" gate="G$1" pin="9"/>
 <wire x1="81.28" y1="66.04" x2="78.74" y2="66.04" width="0.1524" layer="91"/>
 <label x="81.28" y="66.04" size="1.778" layer="95"/>
+<pinref part="U$2" gate="G$1" pin="+12V"/>
 </segment>
 <segment>
@@
 <net name="-12V_INLET" class="0">
 <segment>
-<pinref part="SV1" gate="G$1" pin="1"/>
 <wire x1="81.28" y1="55.88" x2="78.74" y2="55.88" width="0.1524" layer="91"/>
 <label x="81.28" y="55.88" size="1.778" layer="95"/>
-</segment>
-<segment>
-<pinref part="SV1" gate="G$1" pin="2"/>
-<wire x1="60.96" y1="55.88" x2="63.5" y2="55.88" width="0.1524" layer="91"/>
-<label x="45.72" y="55.88" size="1.778" layer="95"/>
-</segment>
-<segment>
+<pinref part="U$2" gate="G$1" pin="-12V"/>
+</segment>
+<segment>
