File: magnetophone.brd (EAGLE design)
At the start: 99 x 19 mm, 22 parts, among them U1 TL074_

Commit message: double!
Parts:
- added C7: 47uf, SparkFun-Passives:CPOL-RADIAL-10UF-25V
- added C8: 15nf, TomW:C050-024X044
- added GAIN1: 50k, TomW:EVUF
- added R2, R6: 2.2k, TomW:0207/10
- added R3: 220R, TomW:0207/10
- added R4: 200R, TomW:0207/10
- added R5: 200k, TomW:0207/10
- added R7: 3.6k, TomW:0207/10
- added RV1: (no value), SparkFun-Electromechanical:POT_PANASONIC_DUAL_VERT_KIT
- added U$4: MONO_CASSETTE_HEAD, MusicThingModular:MONO_CASSETTE_HEAD
- added U$5, U$6: THONKICONNNEW, MusicThingModular:WQP-PJ301M-12_JACK
- moved C3 88.6 mm to (3.17, 82.5)
- moved C6 88.6 mm to (4.45, 76.2)
- moved R1 88.6 mm to (6.99, 73.0)
- moved GAIN 82.2 mm to (79.4, 74.3)
- moved R16 48.2 mm to (49.5, 48.9)
- moved R12 46.5 mm to (62.2, 49.5)
- moved R14 41.0 mm to (59.1, 41.9)
- moved C5 29.3 mm to (52.1, 40.6)
- moved C4 19.7 mm to (61.6, 29.8)
- moved U$1 19.1 mm to (67.9, 14.6)
Connections:
- new net N$11: U$5.P$1_TIP, U1.10
- new net N$12: GAIN1.2, GAIN1.3, R3.1, U1.14
- new net N$13: R3.2, U$6.P$1_TIP
- new net N$14: R5.1, R7.2, U1.12, U1.8
- new net N$15: C8.2, R4.2, R5.2, U1.9
- new net N$16: R2.2, R6.2, U1.13
- new net N$17: GAIN1.1, R2.1
- new net N$18: U$4.P$1, U$5.P$2_SWITCH
- new net N$19: C7.1, R4.1
- new net N$20: C8.1, R7.1
- net GND: now also C7.2, R6.1, U$4.P$2, U$5.P$3_SLEEVE, U$6.P$3_SLEEVE

Commit message: Starting layout
Parts:
- removed C7: 47uf, SparkFun-Passives:CPOL-RADIAL-10UF-25V
- removed C8: 15nf, TomW:C050-024X044
- removed GAIN1: 50k, TomW:EVUF
- removed R2, R6: 2.2k, TomW:0207/10
- removed R3: 220R, TomW:0207/10
- removed R4: 200R, TomW:0207/10
- removed R5: 200k, TomW:0207/10
- removed R7: 3.6k, TomW:0207/10
- removed RV1: (no value), SparkFun-Electromechanical:POT_PANASONIC_DUAL_VERT_KIT
- removed U$2, U$5, U$6: THONKICONNNEW, MusicThingModular:WQP-PJ301M-12_JACK
- removed U$4: MONO_CASSETTE_HEAD, MusicThingModular:MONO_CASSETTE_HEAD
- removed U1: TL074_, MusicThingModular:DIL14
- added OUT: THONKICONNNEW, MusicThingModular:WQP-PJ301M-12_JACK
- added U2: TL072_, MusicThingModular:DIL08
- R1, R10, R12, R14, R16, R8: device TomW:0207/10 -> MusicThingModular:7MM_RESISTOR
- moved C3 92.8 mm to (50.2, 2.54)
- moved C6 83.8 mm to (55.2, 9.53), turned to 90 degrees
- moved GAIN 82.7 mm to (27.9, 9.53)
- moved R1 81.3 mm to (57.8, 9.53), turned to 90 degrees
- moved R14 52.0 mm to (18.4, 9.53), turned to 270 degrees
- moved R16 51.8 mm to (15.9, 9.53), turned to 90 degrees
- moved R12 48.4 mm to (34.9, 9.53), turned to 90 degrees
- moved C5 34.4 mm to (37.5, 9.53)
- moved C4 23.3 mm to (50.2, 9.53)
- moved R10 10.6 mm to (60.3, 9.53)
- moved U$1 9.69 mm to (76.2, 9.53)
- moved 1 6.98 mm to (95.9, 5.08)
- moved C1 6.98 mm to (88.3, 2.54)
- moved C2 6.98 mm to (88.9, 15.9)
- moved D5 6.98 mm to (98.4, 2.54)
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- renumbered U$3 to EXT
Connections:
- removed net N$11: U$5.P$1_TIP, U1.10
- removed net N$12: GAIN1.2, GAIN1.3, R3.1, U1.14
- removed net N$13: R3.2, U$6.P$1_TIP
- removed net N$14: R5.1, R7.2, U1.12, U1.8
- removed net N$15: C8.2, R4.2, R5.2, U1.9
- removed net N$16: R2.2, R6.2, U1.13
- removed net N$17: GAIN1.1, R2.1
- removed net N$18: U$4.P$1, U$5.P$2_SWITCH
- removed net N$19: C7.1, R4.1
- removed net N$20: C8.1, R7.1
- net +12V: now also U2.8; no longer U1.4
- net -12V: now also U2.4; no longer U1.11
- net GND: now also OUT.P$3_SLEEVE, R12.2; no longer C7.2, R12.1, R6.1, U$2.P$3_SLEEVE, U$4.P$2, U$5.P$3_SLEEVE, U$6.P$3_SLEEVE
- net N$1: now also EXT.P$2_SWITCH; no longer U$2.P$2_SWITCH
- net N$10: now also OUT.P$1_TIP; no longer EXT.P$1_TIP
- net N$2: now also EXT.P$1_TIP, U2.3; no longer U$2.P$1_TIP, U1.3
- net N$3: now also R10.1, R8.1, U2.2; no longer R10.2, R8.2, U1.2
- net N$4: now also R10.2, U2.1, U2.5; no longer R10.1, U1.1, U1.5
- net N$6: now also R12.1, U2.6; no longer R12.2, U1.6
- net N$7: now also R8.2; no longer R8.1
- net N$8: now also U2.7; no longer U1.7
Other:
- board size 99 x 19 mm -> 105 x 19 mm

Commit message: First pcb layout
Parts:
- removed SV1: (no value), TomW:MA05-2
- added U$2: EURO_POWER_LOCK, MusicThingModular:EURO_PWR_HEADER_LOCK
- moved R12 18.5 mm to (17.8, 16.5), turned to 0 degrees
- moved C3 17.6 mm to (61.6, 15.9)
- moved C5 16.5 mm to (52.1, 17.1), turned to 180 degrees
- moved EXT 16.1 mm to (21.6, 9.53)
- moved GAIN 13.3 mm to (41.3, 9.53)
- moved R14 12.9 mm to (29.2, 16.5), turned to 0 degrees
- moved R16 12.3 mm to (5.71, 16.5), turned to 0 degrees
- moved R1 10.3 mm to (67.3, 5.71)
- moved C6 10.3 mm to (64.8, 5.71)
- moved R8 10.3 mm to (62.2, 5.71)
- moved R10 10.3 mm to (69.8, 5.71)
- moved U2 9.53 mm to (53.3, 9.53)
- moved C4 8.82 mm to (54.6, 1.91), turned to 180 degrees
- moved OUT 5.08 mm to (6.35, 9.53)
- moved U$1 3.12 mm to (79.3, 9.53)
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Connections:
- net +12V_INLET: now also U$2.POS1, U$2.POS2; no longer SV1.10, SV1.9
- net -12V: now also C5.1; no longer C5.2
- net -12V_INLET: now also U$2.NEG1, U$2.NEG2; no longer SV1.1, SV1.2
- net GND: now also C5.2, R12.1, U$2.GND1, U$2.GND2, U$2.GND3, U$2.GND4, U$2.GND5, U$2.GND6; no longer C5.1, R12.2, SV1.3, SV1.4, SV1.5, SV1.6, SV1.7, SV1.8
- net N$10: now also R16.1; no longer R16.2
- net N$6: now also R12.2; no longer R12.1
- net N$8: now also R16.2; no longer R16.1
Routing:
- net N$1: track 0.00 -> 63.3 mm
- net N$8: track 0.00 -> 52.3 mm
- net -12V: track 0.00 -> 48.0 mm
- net +12V: track 0.00 -> 42.4 mm
- net N$2: track 0.00 -> 39.7 mm
- net N$6: track 0.00 -> 37.6 mm
- net N$3: track 0.00 -> 28.7 mm
- net N$4: track 0.00 -> 25.8 mm
- net +12V_INLET: track 0.00 -> 15.8 mm
- net -12V_INLET: track 0.00 -> 14.4 mm
- net N$5: track 0.00 -> 10.7 mm
- net N$10: track 0.00 -> 7.21 mm
- net N$7: track 0.00 -> 6.61 mm
- net N$9: track 0.00 -> 3.07 mm
Other:
- outline, holes or cut-outs redrawn
- board text added: "Cut out"

Commit message: panel design
Parts:
- turned U$2 to 180 degrees
Routing:
- net N$8: track 52.3 -> 61.7 mm
- net N$2: track 39.7 -> 44.9 mm
- net N$4: track 25.8 -> 28.0 mm
- net -12V_INLET: track 14.4 -> 16.2 mm
- net +12V_INLET: track 15.8 -> 14.4 mm
- net N$1: track 63.3 -> 64.7 mm
- net N$6: track 37.6 -> 38.9 mm
