File: magnetophone_panel.brd (EAGLE design)
At the start: 128.5 x 20 mm, 0 parts

Commit message: panel design
Routing:
- net N$4: track 0.00 -> 50.1 mm
- net N$3: track 0.00 -> 44.5 mm
- net N$2: track 0.00 -> 42.7 mm
- net N$5: track 0.00 -> 35.1 mm
- net N$1: track 0.00 -> 34.6 mm
- net N$6: track 0.00 -> 32.0 mm
