File: Hardware/magnetophone.sch (EAGLE design)
At the start: 22 parts, among them U2 TL072_

Commit message: Tweaks
Parts:
- R16: value 220R -> 200R
Changed lines of the file:
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@@
 <?xml version="1.0" encoding="utf-8"?>
 <!DOCTYPE eagle SYSTEM "eagle.dtd">
-<eagle version="7.4.0">
+<eagle version="7.2.0">
 <drawing>
 <settings>
@@
 <part name="SUPPLY3" library="supply2" deviceset="GND" device=""/>
 <part name="R14" library="MusicThingModular" deviceset="RESISTOR" device="7MM" value="2.2k"/>
-<part name="R16" library="MusicThingModular" deviceset="RESISTOR" device="7MM" value="220R"/>
+<part name="R16" library="MusicThingModular" deviceset="RESISTOR" device="7MM" value="200R"/>
 <part name="SUPPLY7" library="supply2" deviceset="GND" device=""/>
 <part name="R8" library="MusicThingModular" deviceset="RESISTOR" device="7MM" value="200R"/>
