File: Hardware/Magnetophon.brd (EAGLE design)
At the start: 105 x 19 mm, 23 parts, among them U2 TL072_

Commit message: update R12 to improve gain
Parts:
- R12: value 2.2k -> 470R
Changed lines of the file:
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@@
 <element name="R8" library="MusicThingModular" package="7MM_RESISTOR" value="200R" x="60.325" y="6.35" rot="R90"/>
 <element name="R10" library="MusicThingModular" package="7MM_RESISTOR" value="200k" x="65.405" y="6.35" rot="R90"/>
-<element name="R12" library="MusicThingModular" package="7MM_RESISTOR" value="2.2k" x="17.78" y="16.51"/>
+<element name="R12" library="MusicThingModular" package="7MM_RESISTOR" value="470R" x="17.78" y="16.51"/>
 <element name="C1" library="SparkFun-Passives" package="CPOL-RADIAL-10UF-25V" value="10uf" x="88.9" y="2.54" smashed="yes" rot="R180">
 <attribute name="NAME" x="86.614" y="1.3335" size="1.016" layer="25" rot="R180"/>

Commit message: Reroute to avoid space under socket
Routing:
- net N$8: track 54.2 -> 59.5 mm
